File: Ravanesh.kicad_sch (KiCad schematic)
At the start: 23 parts, among them IC1 SPX3819M5-L-5-0_TR, J1 Header_Shrouded_2vias, J2 Conn_01x19_Socket, J3 Conn_01x19_Socket, J5 440054-5, Q1 BC817, Q2 BC817, SW1 SW_Push, SW2 SW_Push, U1 TPS76733QPWPG4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

Commit message: update
Parts:
- added C10: 100nF, Capacitor_SMD:C_0603_1608Metric, symbol Device:C
- added C9: 10uF, Capacitor_SMD:C_0603_1608Metric, symbol Device:C
- added Q3: 2N7000, Package_TO_SOT_THT:TO-92_Inline, symbol Transistor_FET:2N7000
- added R4: 10K, Resistor_SMD:R_0805_2012Metric, symbol Device:R
- added R5: 220, symbol Device:R
Connections:
- net +3V3: now also C10.2, C9.2, R4.2
- net EN: now also R4.1
- net GND: now also C10.1, C9.1
- new net: Q3.2 (G), R5.2
- new net Earth: Q3.1 (S), Q3.3 (D)
- new net MOSFET_GND: R5.1
Other:
- note added: "0,130V Nível lógico baixo"
- note added: "100nF"
- note added: "10uF"
- note added: "1nF"
- note added: "1uF"
- note added: "OK"
- note added: "Paralelo"
- note added: "Pull-up (para garantir o nível) 10K"
- moved on the sheet: J2, J3
